File: gatedriver-sim.sch (KiCad schematic (older format))
At the start: 18 parts, among them Q1 AO3400A, Q2 AO3400A, Q3 AO3400A, Q7 MMBT5551, Q8 MMBT5551, Q9 MMBT5401

Commit message: sim works nicely with 3 fets @ 5A, hits >100°C for 10A.  will change mosfet.
Parts:
- removed Q8: MMBT5551, Package_TO_SOT_SMD:SOT-23, symbol Device:Q_NPN_CBE
- removed R1: 1k, Resistor_SMD:R_0402_1005Metric, symbol Device:R
- removed R3: 0.1, Resistor_SMD:R_0402_1005Metric, symbol Device:R
- removed R5: 4.7k, Resistor_SMD:R_0402_1005Metric, symbol Device:R
- C2: value 3.3n -> 100n
- R2: value 120 -> 1k
- R4: value 4.7k -> 100k
- V1: Spice_Model dc(5) -> dc({vgatedrv})
- V2: Spice_Model pulse(0 3.3 0 {pwm_edge} {pwm_edge} {(pwm_duty)/pwm_freq-2*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 -> dc(0) pulse(0 {vlogic} 0 {pwm_edge} {pwm_edge} {(pwm_duty)/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
Connections:
- net PULSE is gone; now on net BASES: V2.1
- net BASES: now also R6.1
- net at V3.1: now also R7.1
Other:
- note added: ".param temp_a=40\n.param tja=125\n.param n_fets=3\n\n.param pwm_freq=240\n.param pwm_duty=0.8\n.param pwm_edge=0.5u\n\n.param vlogic=5\n.param vgatedrv=5\n.param vled=24\n\n.csparam temp_a={temp_a}\n.csparam tja={tja}\n.csparam n_fets={n_fets}\n.csparam pwm_freq={pwm_freq}\n.csparam pwm_duty={pwm_duty}\n.csparam pwm_edge={pwm_edge}\n.csparam vlogic={vlogic}\n.csparam vgatedrv={vgatedrv}\n.csparam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"
- note added: "TODO in schematic\n - rework driver as per this design\n - remove 9v supply, run everything (inc. MCU) off 5v\n - add 3 more power-mosfets to each channel (6 total per channel)"
- note removed: ".param temp_a=50\n.param n_fets=3\n\n.param pwm_freq=1440\n.param pwm_duty=0.15\n.param pwm_edge=10u\n\n.param vled=24\n\n.csparam temp_a={temp_a}\n.csparam n_fets={n_fets}\n.csparam pwm_freq={pwm_freq}\n.csparam pwm_duty={pwm_duty}\n.csparam pwm_edge={pwm_edge}\n.csparam vled={vled}\n\n.options savecurrents\n.option temp='temp_a'\n.tran 1u {3/pwm_freq}\n\n.control\n\nlet temp_a=$&temp_a\nlet n_f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"
- note removed: "Fixes:\n - Q11 col-resistors act as divider, idiot\n - gate pulldown resistor pulls down too hard?\n - gate RC\n - pwm freq\n - can run off 5v with decent perf (as can the MCU)\n -"
- moved on the sheet: C1, C2, R2, R4, R7, V3

Commit message: lets try a single irlr7843 instead
Parts:
- removed R4: 100k, Resistor_SMD:R_0402_1005Metric, symbol Device:R
- added C3: 100n, Capacitor_SMD:C_0402_1005Metric, symbol Device:C
- Q1, Q2, Q3: value AO3400A -> NTMS4807N; Spice_Lib_File spice/AO3400.mod -> spice/NTMS4807NR2G.LIB; Spice_Model AO3400 -> ntms4807nr2g
- R2: value 1k -> 4.7k
- R7: value 2.4 -> {vled/iled}
Connections:
- net 0: now also C3.2
- net GATE: now also C3.1
Other:
- note added: ".param temp_a=40\n.param tja=80.5\n.param n_fets=3\n\n.param pwm_freq=240\n.param pwm_duty=0.8\n.param pwm_edge=0.5u\n\n.param vlogic=5\n.param vgatedrv=5\n.param vled=24\n.param iled=8\n\n.csparam temp_a={temp_a}\n.csparam tja={tja}\n.csparam n_fets={n_fets}\n.csparam pwm_freq={pwm_freq}\n.csparam pwm_duty={pwm_duty}\n.csparam pwm_edge={pwm_edge}\n.csparam vlogic={vlogic}\n.csparam vgatedrv={vga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"
- note removed: ".param temp_a=40\n.param tja=125\n.param n_fets=3\n\n.param pwm_freq=240\n.param pwm_duty=0.8\n.param pwm_edge=0.5u\n\n.param vlogic=5\n.param vgatedrv=5\n.param vled=24\n\n.csparam temp_a={temp_a}\n.csparam tja={tja}\n.csparam n_fets={n_fets}\n.csparam pwm_freq={pwm_freq}\n.csparam pwm_duty={pwm_duty}\n.csparam pwm_edge={pwm_edge}\n.csparam vlogic={vlogic}\n.csparam vgatedrv={vgatedrv}\n.csparam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"
- note removed: "10A@24V = 2.4Ω effective load"

Commit message: sim with irlr7843
Parts:
- removed C3: 100n, Capacitor_SMD:C_0402_1005Metric, symbol Device:C
- removed Q3: NTMS4807N, Package_TO_SOT_SMD:SOT-23, symbol Transistor_FET:AO3400A
- Q1, Q2: value NTMS4807N -> IRLR7843; Spice_Lib_File spice/NTMS4807NR2G.LIB -> spice/irlru7843.spi.lib; Spice_Model ntms4807nr2g -> irlru7843
- V2: Spice_Model dc(0) pulse(0 {vlogic} 0 {pwm_edge} {pwm_edge} {(pwm_duty)/pwm_freq-2*pwm_edge} {1/pwm_freq} -1) -> dc(0) pulse(0 {vlogic} 0 {pwm_edge} {pwm_edge} {(pwm_duty)/pwm_freq-pwm_edge} {1/pwm_freq} -1)
Other:
- note added: ".param temp_a=40\n.param tja=50\n.param n_fets=2\n\n.param pwm_freq=240\n.param pwm_duty=0.8\n.param pwm_edge=0.5u\n\n.param vlogic=5\n.param vgatedrv=5\n.param vled=24\n.param iled=8\n\n.csparam temp_a={temp_a}\n.csparam tja={tja}\n.csparam n_fets={n_fets}\n.csparam pwm_freq={pwm_freq}\n.csparam pwm_duty={pwm_duty}\n.csparam pwm_edge={pwm_edge}\n.csparam vlogic={vlogic}\n.csparam vgatedrv={vgate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"
- note removed: ".param temp_a=40\n.param tja=80.5\n.param n_fets=3\n\n.param pwm_freq=240\n.param pwm_duty=0.8\n.param pwm_edge=0.5u\n\n.param vlogic=5\n.param vgatedrv=5\n.param vled=24\n.param iled=8\n\n.csparam temp_a={temp_a}\n.csparam tja={tja}\n.csparam n_fets={n_fets}\n.csparam pwm_freq={pwm_freq}\n.csparam pwm_duty={pwm_duty}\n.csparam pwm_edge={pwm_edge}\n.csparam vlogic={vlogic}\n.csparam vgatedrv={vga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"

Commit message: happy with driver design, migrate back to schematic
Parts:
- added Q3: NTMS4807, symbol Transistor_FET:AO3400A
- C2: value 100n -> 3.3n
- Q1, Q2: value IRLR7843 -> NTMS4807; footprint Package_TO_SOT_SMD:SOT-23 -> (none); JLC C20917 -> (none); Spice_Lib_File spice/irlru7843.spi.lib -> spice/NTMS4807NR2G.LIB; Spice_Model irlru7843 -> ntms4807nr2g
Connections:
- net 0: now also Q3.2 (S)
- net DRAIN: now also Q3.3 (D)
- net GATE: now also Q3.1 (G)
Other:
- note added: ".param temp_a=40\n.param tja=80.5\n.param n_fets=3\n\n.param pwm_freq=240\n.param pwm_duty=0.5\n.param pwm_edge=0.5u\n\n.param vlogic=5\n.param vgatedrv=5\n.param vled=24\n.param iled=8\n\n.param sim_periods=5\n\n.csparam temp_a={temp_a}\n.csparam tja={tja}\n.csparam n_fets={n_fets}\n.csparam pwm_freq={pwm_freq}\n.csparam pwm_duty={pwm_duty}\n.csparam pwm_edge={pwm_edge}\n.csparam vlogic={vlogic}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"
- note added: "B = μ₀ I / 2πr\n\nμ₀ = 2αh/e²c = 1.3e-6 m kg s¯² A¯²\n\ndB/dt = μ₀ dI/dt / 2πr = 2e-7 dI/dt / r"
- note added: "https://scantech7.com/emf-rf-magnetic-electric-field-sound-noise-radiation-safety-levels-dallas-fort-worth-houston-austin/"
- note removed: ".param temp_a=40\n.param tja=50\n.param n_fets=2\n\n.param pwm_freq=240\n.param pwm_duty=0.8\n.param pwm_edge=0.5u\n\n.param vlogic=5\n.param vgatedrv=5\n.param vled=24\n.param iled=8\n\n.csparam temp_a={temp_a}\n.csparam tja={tja}\n.csparam n_fets={n_fets}\n.csparam pwm_freq={pwm_freq}\n.csparam pwm_duty={pwm_duty}\n.csparam pwm_edge={pwm_edge}\n.csparam vlogic={vlogic}\n.csparam vgatedrv={vgate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"

Commit message: ready?
Parts:
- removed Q3: NTMS4807, symbol Transistor_FET:AO3400A
Other:
- note added: ".param temp_a=40\n.param tja=80.5\n.param n_fets=2\n\n.param pwm_freq=240\n.param pwm_duty=0.5\n.param pwm_edge=0.5u\n\n.param vlogic=5\n.param vgatedrv=5\n.param vled=24\n.param iled=8\n\n.param sim_periods=5\n\n.csparam temp_a={temp_a}\n.csparam tja={tja}\n.csparam n_fets={n_fets}\n.csparam pwm_freq={pwm_freq}\n.csparam pwm_duty={pwm_duty}\n.csparam pwm_edge={pwm_edge}\n.csparam vlogic={vlogic}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"
- note removed: ".param temp_a=40\n.param tja=80.5\n.param n_fets=3\n\n.param pwm_freq=240\n.param pwm_duty=0.5\n.param pwm_edge=0.5u\n\n.param vlogic=5\n.param vgatedrv=5\n.param vled=24\n.param iled=8\n\n.param sim_periods=5\n\n.csparam temp_a={temp_a}\n.csparam tja={tja}\n.csparam n_fets={n_fets}\n.csparam pwm_freq={pwm_freq}\n.csparam pwm_duty={pwm_duty}\n.csparam pwm_edge={pwm_edge}\n.csparam vlogic={vlogic}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"
Changed lines of the file:
@@
 	3250 1200 4000 1200
 Text Notes 11800 10950 0    39   ~ 0
-.param temp_a=40\n.param tja=80.5\n.param n_fets=3\n\n.param pwm_freq=240\n.param pwm_duty=0.5\n.param pwm_edge=0.5u\n\n.param vlogic=5\n.param vgatedrv=5\n.param vled=24\n.param iled=8\n\n.param sim_periods=5\n\n.csparam temp_a={temp_a}\n.csparam tja={tja}\n.csparam n_fets={n_fets}\n.csparam pwm_freq={pwm_freq}\n.csparam pwm_duty={pwm_duty}\n.csparam pwm_edge={pwm_edge}\n.csparam vlogic={vlogic}\n.csparam vgatedrv={vgatedrv}\n.csparam vled={vled}\n.csparam iled={iled}\n.csparam sim_periods={sim_periods}\n\n.options savecurrents\n.option temp='temp_a'\n\n.tran {1/2048/pwm_freq} {sim_periods/pwm_freq}\n\n.control\n\npre_set strict_errorhandling\n\nlet temp_a=$&temp_a\nlet n_fets=$&n_fets\nlet tja=$&tja\nlet pwm_freq=$&pwm_freq\nlet pwm_duty=$&pwm_duty\nlet pwm_edge=$&pwm_edge\nlet vlogic=$&vlogic\nlet vgatedrv=$&vgatedrv\nlet vled=$&vled\nlet iled=$&iled\nlet sim_periods=$&sim_periods\n\nlet id=@R7[i]\nlet vd=v("/DRAIN")\nlet pds=vd*id\n\nmeas TRAN id_min MIN id\nmeas TRAN id_max MAX id\nlet idl=0.1*(id_max-id_min)+id_min\nlet idh=0.9*(id_max-id_min)+id_min\n\nmeas TRAN id_rise_time TRIG id VAL=idl RISE=2 TARG id VAL=idh RISE=2\nmeas TRAN id_fall_time TRIG id VAL=idh FALL=2 TARG id VAL=idl FALL=2\n\nmeas TRAN id_rise_from WHEN id=idl RISE=2\nmeas TRAN id_rise_to WHEN id=idh RISE=1 td=id_rise_from\nmeas TRAN id_fall_from WHEN id=idh FALL=1 td=id_rise_to\nmeas TRAN id_fall_to WHEN id=idl FALL=1 td=id_fall_from\nmeas TRAN id_rise_from2 WHEN id=idl RISE=2 td=id_fall_to\n\nlet switching_time_fraction=((id_rise_to-id_rise_from)+(id_fall_to-id_fall_from)) / (id_rise_from2-id_rise_from)\n\nmeas tran wds_rise integ pds from=id_rise_from to=id_rise_to\nmeas tran wds_high integ pds from=id_rise_to to=id_fall_from\nmeas tran wds_fall integ pds from=id_fall_from to=id_fall_to\nmeas tran wds_low integ pds from=id_fall_to to=id_rise_from2\nmeas tran wds_all integ pds from=id_rise_from to=id_rise_from2\n\nlet pds_rise=wds_rise/(id_rise_to-id_rise_from)\nlet pds_high=wds_high/(id_fall_from-id_rise_to)\nlet pds_fall=wds_fall/(id_fall_to-id_fall_from)\nlet pds_low=wds_low/(id_rise_from2-id_fall_to)\nlet pds_all=wds_all/(id_rise_from2-id_rise_from)\n\nlet switching_loss=(wds_rise+wds_fall)/wds_all\nlet total_loss=mean(vd*id) / mean((vled-vd)*id)\n\nlet rds=vd/id\nmeas tran rds_on avg rds from=id_rise_to to=id_fall_from\nmeas tran rds_off avg rds from=id_fall_to to=id_rise_from2\n\nlet temp_ja=tja*pds_all/n_fets\nlet temp_j=temp_a+temp_ja\n\nlet i_gpio_max=maximum(@V2[i])\n\necho .\necho CONFIG:\nprint sim_periods\necho .\n\necho Voltages\nprint vlogic\nprint vgatedrv\nprint vled\nprint iled\necho .\n\necho PWM configuration\nprint pwm_freq\nprint pwm_duty\nprint pwm_edge\necho .\n\necho Number of parallel'd transistors\nprint n_fets\necho .\n\necho .\necho RESULTS:\necho .\n\necho Power lost in transistors during rise/high/fall/low\nprint pds_rise\nprint pds_high\nprint pds_fall\nprint pds_low\nprint pds_all\necho .\n\necho Effective Rds(on/off)\nprint rds_on\nprint rds_off\necho .\n\necho Actual Rds(on/off)\nprint rds_on*n_fets\nprint rds_off*n_fets\necho .\n\necho Switching loss as fraction of loss in transistors\nprint switching_loss\necho .\n\necho Loss in transistors as fraction of total power (lost + delivered to load)\nprint total_loss\necho .\n\necho Drain current rise/fall root-frequencies (1/t)\nprint (1/id_rise_time)\nprint (1/id_fall_time)\necho .\n\necho Temperatures\nprint temp_ja\nprint temp_a\nprint temp_j\necho .\n\necho Switching time fraction of full cycle\nprint switching_time_fraction\necho .\n\necho Max GPIO loading\nprint i_gpio_max\necho .\n\nset hcopydevtype=svg\nset svg_intopts=( 1200 900 24 0 1 4 1 )\nsetcs svg_stropts=( black Arial Arial )\nset color1=cyan\nset color2=green\n\nhardcopy sim_ids_tran.svg id title 'Ids transient' xlabel 'Time' ylabel 'Ids'\n\nlinearize id\nset specwindow=none\nfft id\nhardcopy sim_ids_fft.svg db(id) title 'Ids spectrum' xlabel 'Frequency' ylabel 'Ids (db A)'\n\n.endc\n
+.param temp_a=40\n.param tja=80.5\n.param n_fets=2\n\n.param pwm_freq=240\n.param pwm_duty=0.5\n.param pwm_edge=0.5u\n\n.param vlogic=5\n.param vgatedrv=5\n.param vled=24\n.param iled=8\n\n.param sim_periods=5\n\n.csparam temp_a={temp_a}\n.csparam tja={tja}\n.csparam n_fets={n_fets}\n.csparam pwm_freq={pwm_freq}\n.csparam pwm_duty={pwm_duty}\n.csparam pwm_edge={pwm_edge}\n.csparam vlogic={vlogic}\n.csparam vgatedrv={vgatedrv}\n.csparam vled={vled}\n.csparam iled={iled}\n.csparam sim_periods={sim_periods}\n\n.options savecurrents\n.option temp='temp_a'\n\n.tran {1/2048/pwm_freq} {sim_periods/pwm_freq}\n\n.control\n\npre_set strict_errorhandling\n\nlet temp_a=$&temp_a\nlet n_fets=$&n_fets\nlet tja=$&tja\nlet pwm_freq=$&pwm_freq\nlet pwm_duty=$&pwm_duty\nlet pwm_edge=$&pwm_edge\nlet vlogic=$&vlogic\nlet vgatedrv=$&vgatedrv\nlet vled=$&vled\nlet iled=$&iled\nlet sim_periods=$&sim_periods\n\nlet id=@R7[i]\nlet vd=v("/DRAIN")\nlet pds=vd*id\n\nmeas TRAN id_min MIN id\nmeas TRAN id_max MAX id\nlet idl=0.1*(id_max-id_min)+id_min\nlet idh=0.9*(id_max-id_min)+id_min\n\nmeas TRAN id_rise_time TRIG id VAL=idl RISE=2 TARG id VAL=idh RISE=2\nmeas TRAN id_fall_time TRIG id VAL=idh FALL=2 TARG id VAL=idl FALL=2\n\nmeas TRAN id_rise_from WHEN id=idl RISE=2\nmeas TRAN id_rise_to WHEN id=idh RISE=1 td=id_rise_from\nmeas TRAN id_fall_from WHEN id=idh FALL=1 td=id_rise_to\nmeas TRAN id_fall_to WHEN id=idl FALL=1 td=id_fall_from\nmeas TRAN id_rise_from2 WHEN id=idl RISE=2 td=id_fall_to\n\nlet switching_time_fraction=((id_rise_to-id_rise_from)+(id_fall_to-id_fall_from)) / (id_rise_from2-id_rise_from)\n\nmeas tran wds_rise integ pds from=id_rise_from to=id_rise_to\nmeas tran wds_high integ pds from=id_rise_to to=id_fall_from\nmeas tran wds_fall integ pds from=id_fall_from to=id_fall_to\nmeas tran wds_low integ pds from=id_fall_to to=id_rise_from2\nmeas tran wds_all integ pds from=id_rise_from to=id_rise_from2\n\nlet pds_rise=wds_rise/(id_rise_to-id_rise_from)\nlet pds_high=wds_high/(id_fall_from-id_rise_to)\nlet pds_fall=wds_fall/(id_fall_to-id_fall_from)\nlet pds_low=wds_low/(id_rise_from2-id_fall_to)\nlet pds_all=wds_all/(id_rise_from2-id_rise_from)\n\nlet switching_loss=(wds_rise+wds_fall)/wds_all\nlet total_loss=mean(vd*id) / mean((vled-vd)*id)\n\nlet rds=vd/id\nmeas tran rds_on avg rds from=id_rise_to to=id_fall_from\nmeas tran rds_off avg rds from=id_fall_to to=id_rise_from2\n\nlet temp_ja=tja*pds_all/n_fets\nlet temp_j=temp_a+temp_ja\n\nlet i_gpio_max=maximum(@V2[i])\n\necho .\necho CONFIG:\nprint sim_periods\necho .\n\necho Voltages\nprint vlogic\nprint vgatedrv\nprint vled\nprint iled\necho .\n\necho PWM configuration\nprint pwm_freq\nprint pwm_duty\nprint pwm_edge\necho .\n\necho Number of parallel'd transistors\nprint n_fets\necho .\n\necho .\necho RESULTS:\necho .\n\necho Power lost in transistors during rise/high/fall/low\nprint pds_rise\nprint pds_high\nprint pds_fall\nprint pds_low\nprint pds_all\necho .\n\necho Effective Rds(on/off)\nprint rds_on\nprint rds_off\necho .\n\necho Actual Rds(on/off)\nprint rds_on*n_fets\nprint rds_off*n_fets\necho .\n\necho Switching loss as fraction of loss in transistors\nprint switching_loss\necho .\n\necho Loss in transistors as fraction of total power (lost + delivered to load)\nprint total_loss\necho .\n\necho Drain current rise/fall root-frequencies (1/t)\nprint (1/id_rise_time)\nprint (1/id_fall_time)\necho .\n\necho Temperatures\nprint temp_ja\nprint temp_a\nprint temp_j\necho .\n\necho Switching time fraction of full cycle\nprint switching_time_fraction\necho .\n\necho Max GPIO loading\nprint i_gpio_max\necho .\n\nset hcopydevtype=svg\nset svg_intopts=( 1200 900 24 0 1 4 1 )\nsetcs svg_stropts=( black Arial Arial )\nset color1=cyan\nset color2=green\n\nhardcopy sim_ids_tran.svg id title 'Ids transient' xlabel 'Time' ylabel 'Ids'\n\nlinearize id\nset specwindow=none\nfft id\nhardcopy sim_ids_fft.svg db(id) title 'Ids spectrum' xlabel 'Frequency' ylabel 'Ids (db A)'\n\n.endc\n
 Wire Wire Line
 	5450 2000 6750 2000
@@
 Connection ~ 2250 4000
 Wire Wire Line
-	2250 4000 3000 4000
-$Comp
-L Transistor_FET:AO3400A Q?
-U 1 1 61D1ACC7
-P 2900 4200
-AR Path="/61B5C5B6/61D1ACC7" Ref="Q?"  Part="1"
-AR Path="/61C03040/61D1ACC7" Ref="Q?"  Part="1"
-AR Path="/61C031A1/61D1ACC7" Ref="Q?"  Part="1"
-AR Path="/61C031A3/61D1ACC7" Ref="Q?"  Part="1"
-AR Path="/61D1ACC7" Ref="Q3"  Part="1"
-AR Path="/6202E846/61D1ACC7" Ref="Q?"  Part="1"
-AR Path="/620593AE/61D1ACC7" Ref="Q?"  Part="1"
-F 0 "Q3" H 3105 4246 50  0000 L CNN
-F 1 "NTMS4807" H 3105 4155 50  0000 L CNN
-F 2 "" H 3100 4125 50  0001 L CIN
-F 3 "" H 2900 4200 50  0001 L CNN
-F 4 "X" H 2900 4200 50  0001 C CNN "Spice_Primitive"
-F 5 "ntms4807nr2g" H 2900 4200 50  0001 C CNN "Spice_Model"
-F 6 "Y" H 2900 4200 50  0001 C CNN "Spice_Netlist_Enabled"
-F 7 "spice/NTMS4807NR2G.LIB" H 2900 4200 50  0001 C CNN "Spice_Lib_File"
-F 8 "3 1 2" H 2900 4200 50  0001 C CNN "Spice_Node_Sequence"
-	1    2900 4200
-	1    0    0    -1
-$EndComp
-Wire Wire Line
 	1150 4200 1950 4200
 Wire Wire Line
 	1450 4400 2250 4400
-Connection ~ 2250 4400
-Wire Wire Line
-	2250 4400 3000 4400
-Connection ~ 1950 4200
-Wire Wire Line
-	1950 4200 2700 4200
-Connection ~ 3000 4000
-Wire Wire Line
-	3000 4000 6600 4000
 Text Notes 9350 6300 0    50   ~ 0
 B = μ₀ I / 2πr\n\nμ₀ = 2αh/e²c = 1.3e-6 m kg s¯² A¯²\n\ndB/dt = μ₀ dI/dt / 2πr = 2e-7 dI/dt / r
 Text Notes 1100 6500 0    50   ~ 0
 https://scantech7.com/emf-rf-magnetic-electric-field-sound-noise-radiation-safety-levels-dallas-fort-worth-houston-austin/
+Wire Wire Line
+	2250 4000 6600 4000
 $EndSCHEMATC

Commit message: we can tolerate higher frequencies as long as our led strips are only a dozen or so metres long
Parts:
- removed Q2: NTMS4807, symbol Transistor_FET:AO3400A
- C2: value 3.3n -> 100n
- Q1: value NTMS4807 -> SiS402; Spice_Lib_File spice/NTMS4807NR2G.LIB -> spice/SiS402DN_PS.lib; Spice_Model ntms4807nr2g -> SiS402DN
- R2: value 4.7k -> 220
Other:
- note added: ".param temp_a=40\n\n* https://datasheet.lcsc.com/lcsc/1809301517_Vishay-Intertech-SIS402DN-T1-GE3_C15791.pdf p11\n.param tja=70\n.param tjc=2.4\n\n.param n_fets=1\n\n.param pwm_freq=240\n.param pwm_duty=0.5\n.param pwm_edge=0.5u\n\n.param vlogic=5\n.param vgatedrv=5\n.param vled=24\n.param iled=8\n\n.param sim_periods=5\n\n.csparam temp_a={temp_a}\n.csparam tja={tja}\n.csparam tjc={tjc}\n.csparam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"
- note removed: ".param temp_a=40\n.param tja=80.5\n.param n_fets=2\n\n.param pwm_freq=240\n.param pwm_duty=0.5\n.param pwm_edge=0.5u\n\n.param vlogic=5\n.param vgatedrv=5\n.param vled=24\n.param iled=8\n\n.param sim_periods=5\n\n.csparam temp_a={temp_a}\n.csparam tja={tja}\n.csparam n_fets={n_fets}\n.csparam pwm_freq={pwm_freq}\n.csparam pwm_duty={pwm_duty}\n.csparam pwm_edge={pwm_edge}\n.csparam vlogic={vlogic}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"
- note removed: "B = μ₀ I / 2πr\n\nμ₀ = 2αh/e²c = 1.3e-6 m kg s¯² A¯²\n\ndB/dt = μ₀ dI/dt / 2πr = 2e-7 dI/dt / r"
- note removed: "TODO in schematic\n - rework driver as per this design\n - remove 9v supply, run everything (inc. MCU) off 5v\n - add 3 more power-mosfets to each channel (6 total per channel)"
- moved on the sheet: R7, V3
