File: channel.sch (KiCad schematic (older format))
At the start: 8 parts, among them Q1 MMBT5551, Q2 SiS402DN, Q3 SiS402DN, Q4 MMBT5401

Commit message: swapped placement for 5V LDO vs LEDs, for more stable 5V supply when power-side of ground is noisy
Parts:
- renumbered R9 to R11, R10 to R12
Other:
- note added: "Could just use 3x AO3400 per-channel for a fraction of the cost (also "basic part" on JLC).\n5A per mosfet.\nMuch higher Rds(on) though 32mΩ vs 8mΩ."
- note removed: "TODO\nDouble up the mosfets, since we get charged for min.15 of them anyway."
Changed lines of the file:
@@
 AR Path="/6202E846/61C0AE1D" Ref="#PWR031"  Part="1"
 AR Path="/620593AE/61C0AE1D" Ref="#PWR037"  Part="1"
-F 0 "#PWR031" H 3000 2400 50  0001 C CNN
+F 0 "#PWR037" H 3000 2400 50  0001 C CNN
 F 1 "GND" H 3005 2477 50  0000 C CNN
 F 2 "" H 3000 2650 50  0001 C CNN
@@
 AR Path="/61C031A3/61C0ECF9" Ref="R?"  Part="1"
 AR Path="/61C0ECF9" Ref="R?"  Part="1"
-AR Path="/6202E846/61C0ECF9" Ref="R10"  Part="1"
-AR Path="/620593AE/61C0ECF9" Ref="R12"  Part="1"
-F 0 "R10" H 1530 2646 50  0000 R CNN
+AR Path="/6202E846/61C0ECF9" Ref="R12"  Part="1"
+AR Path="/620593AE/61C0ECF9" Ref="R14"  Part="1"
+F 0 "R14" H 1530 2646 50  0000 R CNN
 F 1 "4.7k" H 1530 2555 50  0000 R CNN
 F 2 "Resistor_SMD:R_0402_1005Metric" V 1530 2600 50  0001 C CNN
@@
 AR Path="/6202E846/61C1051F" Ref="#PWR032"  Part="1"
 AR Path="/620593AE/61C1051F" Ref="#PWR038"  Part="1"
-F 0 "#PWR032" H 1600 2500 50  0001 C CNN
+F 0 "#PWR038" H 1600 2500 50  0001 C CNN
 F 1 "GND" H 1605 2577 50  0000 C CNN
 F 2 "" H 1600 2750 50  0001 C CNN
@@
 AR Path="/6202E846/61C0A1BB" Ref="Q1"  Part="1"
 AR Path="/620593AE/61C0A1BB" Ref="Q5"  Part="1"
-F 0 "Q1" H 3091 1496 50  0000 L CNN
+F 0 "Q5" H 3091 1496 50  0000 L CNN
 F 1 "MMBT5551" H 3091 1405 50  0000 L CNN
 F 2 "Package_TO_SOT_SMD:SOT-23" H 3100 1375 50  0001 L CIN
@@
 AR Path="/61C031A3/61C5A1AF" Ref="R?"  Part="1"
 AR Path="/61C5A1AF" Ref="R?"  Part="1"
-AR Path="/6202E846/61C5A1AF" Ref="R9"  Part="1"
-AR Path="/620593AE/61C5A1AF" Ref="R11"  Part="1"
-F 0 "R9" V 3657 1950 50  0000 C CNN
+AR Path="/6202E846/61C5A1AF" Ref="R11"  Part="1"
+AR Path="/620593AE/61C5A1AF" Ref="R13"  Part="1"
+F 0 "R13" V 3657 1950 50  0000 C CNN
 F 1 "100" V 3566 1950 50  0000 C CNN
 F 2 "Resistor_SMD:R_0402_1005Metric_Pad0.72x0.64mm_HandSolder" V 3380 1950 50  0001 C CNN
@@
 AR Path="/6202E846/61C4E023" Ref="Q4"  Part="1"
 AR Path="/620593AE/61C4E023" Ref="Q8"  Part="1"
-F 0 "Q4" H 3091 2404 50  0000 L CNN
+F 0 "Q8" H 3091 2404 50  0000 L CNN
 F 1 "MMBT5401" H 3091 2495 50  0000 L CNN
 F 2 "Package_TO_SOT_SMD:SOT-23" H 3100 2550 50  0001 C CNN
@@
 AR Path="/6202E846/61D142B7" Ref="C10"  Part="1"
 AR Path="/620593AE/61D142B7" Ref="C12"  Part="1"
-F 0 "C10" H 1265 1346 50  0000 L CNN
+F 0 "C12" H 1265 1346 50  0000 L CNN
 F 1 "100n/50" H 1265 1255 50  0000 L CNN
 F 2 "Capacitor_SMD:C_0402_1005Metric" H 1188 1150 50  0001 C CNN
@@
 AR Path="/6202E846/61D15BBF" Ref="#PWR027"  Part="1"
 AR Path="/620593AE/61D15BBF" Ref="#PWR033"  Part="1"
-F 0 "#PWR027" H 1150 1200 50  0001 C CNN
+F 0 "#PWR033" H 1150 1200 50  0001 C CNN
 F 1 "GND" H 1155 1277 50  0000 C CNN
 F 2 "" H 1150 1450 50  0001 C CNN
@@
 AR Path="/6202E846/622D62B8" Ref="Q2"  Part="1"
 AR Path="/620593AE/622D62B8" Ref="Q6"  Part="1"
-F 0 "Q2" H 5304 1996 50  0000 L CNN
+F 0 "Q6" H 5304 1996 50  0000 L CNN
 F 1 "SiS402DN" H 5304 1905 50  0000 L CNN
 F 2 "Package_SO:Vishay_PowerPAK_1212-8_Single" H 5100 2450 50  0001 C CNN
@@
 AR Path="/6202E846/6203BB32" Ref="#PWR028"  Part="1"
 AR Path="/620593AE/6203BB32" Ref="#PWR034"  Part="1"
-F 0 "#PWR028" H 5200 1900 50  0001 C CNN
+F 0 "#PWR034" H 5200 1900 50  0001 C CNN
 F 1 "GND" H 5205 1977 50  0000 C CNN
 F 2 "" H 5200 2150 50  0001 C CNN
@@
 AR Path="/6202E846/61C61D09" Ref="C11"  Part="1"
 AR Path="/620593AE/61C61D09" Ref="C13"  Part="1"
-F 0 "C11" H 4035 2146 50  0000 R CNN
+F 0 "C13" H 4035 2146 50  0000 R CNN
 F 1 "100n/50" H 4035 2055 50  0000 R CNN
 F 2 "Capacitor_SMD:C_0402_1005Metric_Pad0.74x0.62mm_HandSolder" H 4188 1950 50  0001 C CNN
@@
 AR Path="/6202E846/61C20664" Ref="#PWR030"  Part="1"
 AR Path="/620593AE/61C20664" Ref="#PWR036"  Part="1"
-F 0 "#PWR030" H 4150 2000 50  0001 C CNN
+F 0 "#PWR036" H 4150 2000 50  0001 C CNN
 F 1 "GND" H 4155 2077 50  0000 C CNN
 F 2 "" H 4150 2250 50  0001 C CNN
@@
 	1    0    0    -1
 $EndComp
-Text Notes 3700 2900 0    50   ~ 0
-TODO\nDouble up the mosfets, since we get charged for min.15 of them anyway.
+Text Notes 5000 2700 0    50   ~ 0
+Could just use 3x AO3400 per-channel for a fraction of the cost (also "basic part" on JLC).\n5A per mosfet.\nMuch higher Rds(on) though 32mΩ vs 8mΩ.
 $Comp
 L mark:SiS402DN Q3
@@
 AR Path="/6202E846/6236D64F" Ref="Q3"  Part="1"
 AR Path="/620593AE/6236D64F" Ref="Q7"  Part="1"
-F 0 "Q3" H 6454 1996 50  0000 L CNN
+F 0 "Q7" H 6454 1996 50  0000 L CNN
 F 1 "SiS402DN" H 6454 1905 50  0000 L CNN
 F 2 "Package_SO:Vishay_PowerPAK_1212-8_Single" H 6250 2450 50  0001 C CNN
@@
 AR Path="/6202E846/6236E79F" Ref="#PWR029"  Part="1"
 AR Path="/620593AE/6236E79F" Ref="#PWR035"  Part="1"
-F 0 "#PWR029" H 6350 1900 50  0001 C CNN
+F 0 "#PWR035" H 6350 1900 50  0001 C CNN
 F 1 "GND" H 6355 1977 50  0000 C CNN
 F 2 "" H 6350 2150 50  0001 C CNN

Commit message: order ready
Parts:
- C10, C11: value 100n/50 -> 100n; JLC C307331 -> C1525
Changed lines of the file:
@@
 AR Path="/6202E846/61C0AE1D" Ref="#PWR031"  Part="1"
 AR Path="/620593AE/61C0AE1D" Ref="#PWR037"  Part="1"
-F 0 "#PWR037" H 3000 2400 50  0001 C CNN
+F 0 "#PWR031" H 3000 2400 50  0001 C CNN
 F 1 "GND" H 3005 2477 50  0000 C CNN
 F 2 "" H 3000 2650 50  0001 C CNN
@@
 AR Path="/6202E846/61C0ECF9" Ref="R12"  Part="1"
 AR Path="/620593AE/61C0ECF9" Ref="R14"  Part="1"
-F 0 "R14" H 1530 2646 50  0000 R CNN
+F 0 "R12" H 1530 2646 50  0000 R CNN
 F 1 "4.7k" H 1530 2555 50  0000 R CNN
 F 2 "Resistor_SMD:R_0402_1005Metric" V 1530 2600 50  0001 C CNN
@@
 AR Path="/6202E846/61C1051F" Ref="#PWR032"  Part="1"
 AR Path="/620593AE/61C1051F" Ref="#PWR038"  Part="1"
-F 0 "#PWR038" H 1600 2500 50  0001 C CNN
+F 0 "#PWR032" H 1600 2500 50  0001 C CNN
 F 1 "GND" H 1605 2577 50  0000 C CNN
 F 2 "" H 1600 2750 50  0001 C CNN
@@
 AR Path="/6202E846/61C0A1BB" Ref="Q1"  Part="1"
 AR Path="/620593AE/61C0A1BB" Ref="Q5"  Part="1"
-F 0 "Q5" H 3091 1496 50  0000 L CNN
+F 0 "Q1" H 3091 1496 50  0000 L CNN
 F 1 "MMBT5551" H 3091 1405 50  0000 L CNN
 F 2 "Package_TO_SOT_SMD:SOT-23" H 3100 1375 50  0001 L CIN
@@
 AR Path="/6202E846/61C5A1AF" Ref="R11"  Part="1"
 AR Path="/620593AE/61C5A1AF" Ref="R13"  Part="1"
-F 0 "R13" V 3657 1950 50  0000 C CNN
+F 0 "R11" V 3657 1950 50  0000 C CNN
 F 1 "100" V 3566 1950 50  0000 C CNN
 F 2 "Resistor_SMD:R_0402_1005Metric_Pad0.72x0.64mm_HandSolder" V 3380 1950 50  0001 C CNN
@@
 AR Path="/6202E846/61C4E023" Ref="Q4"  Part="1"
 AR Path="/620593AE/61C4E023" Ref="Q8"  Part="1"
-F 0 "Q8" H 3091 2404 50  0000 L CNN
+F 0 "Q4" H 3091 2404 50  0000 L CNN
 F 1 "MMBT5401" H 3091 2495 50  0000 L CNN
 F 2 "Package_TO_SOT_SMD:SOT-23" H 3100 2550 50  0001 C CNN
@@
 AR Path="/6202E846/61D142B7" Ref="C10"  Part="1"
 AR Path="/620593AE/61D142B7" Ref="C12"  Part="1"
-F 0 "C12" H 1265 1346 50  0000 L CNN
-F 1 "100n/50" H 1265 1255 50  0000 L CNN
+F 0 "C10" H 1265 1346 50  0000 L CNN
+F 1 "100n" H 1265 1255 50  0000 L CNN
 F 2 "Capacitor_SMD:C_0402_1005Metric" H 1188 1150 50  0001 C CNN
 F 3 "~" H 1150 1300 50  0001 C CNN
-F 4 "C307331" H 1150 1300 50  0001 C CNN "JLC"
+F 4 "C1525" H 1150 1300 50  0001 C CNN "JLC"
 	1    1150 1300
 	1    0    0    -1
@@
 AR Path="/6202E846/61D15BBF" Ref="#PWR027"  Part="1"
 AR Path="/620593AE/61D15BBF" Ref="#PWR033"  Part="1"
-F 0 "#PWR033" H 1150 1200 50  0001 C CNN
+F 0 "#PWR027" H 1150 1200 50  0001 C CNN
 F 1 "GND" H 1155 1277 50  0000 C CNN
 F 2 "" H 1150 1450 50  0001 C CNN
@@
 AR Path="/6202E846/622D62B8" Ref="Q2"  Part="1"
 AR Path="/620593AE/622D62B8" Ref="Q6"  Part="1"
-F 0 "Q6" H 5304 1996 50  0000 L CNN
+F 0 "Q2" H 5304 1996 50  0000 L CNN
 F 1 "SiS402DN" H 5304 1905 50  0000 L CNN
 F 2 "Package_SO:Vishay_PowerPAK_1212-8_Single" H 5100 2450 50  0001 C CNN
@@
 AR Path="/6202E846/6203BB32" Ref="#PWR028"  Part="1"
 AR Path="/620593AE/6203BB32" Ref="#PWR034"  Part="1"
-F 0 "#PWR034" H 5200 1900 50  0001 C CNN
+F 0 "#PWR028" H 5200 1900 50  0001 C CNN
 F 1 "GND" H 5205 1977 50  0000 C CNN
 F 2 "" H 5200 2150 50  0001 C CNN
@@
 AR Path="/6202E846/61C61D09" Ref="C11"  Part="1"
 AR Path="/620593AE/61C61D09" Ref="C13"  Part="1"
-F 0 "C13" H 4035 2146 50  0000 R CNN
-F 1 "100n/50" H 4035 2055 50  0000 R CNN
+F 0 "C11" H 4035 2146 50  0000 R CNN
+F 1 "100n" H 4035 2055 50  0000 R CNN
 F 2 "Capacitor_SMD:C_0402_1005Metric_Pad0.74x0.62mm_HandSolder" H 4188 1950 50  0001 C CNN
 F 3 "~" H 4150 2100 50  0001 C CNN
-F 4 "C307331" H 4150 2100 50  0001 C CNN "JLC"
+F 4 "C1525" H 4150 2100 50  0001 C CNN "JLC"
 	1    4150 2100
 	1    0    0    -1
@@
 AR Path="/6202E846/61C20664" Ref="#PWR030"  Part="1"
 AR Path="/620593AE/61C20664" Ref="#PWR036"  Part="1"
-F 0 "#PWR036" H 4150 2000 50  0001 C CNN
+F 0 "#PWR030" H 4150 2000 50  0001 C CNN
 F 1 "GND" H 4155 2077 50  0000 C CNN
 F 2 "" H 4150 2250 50  0001 C CNN
@@
 AR Path="/6202E846/6236D64F" Ref="Q3"  Part="1"
 AR Path="/620593AE/6236D64F" Ref="Q7"  Part="1"
-F 0 "Q7" H 6454 1996 50  0000 L CNN
+F 0 "Q3" H 6454 1996 50  0000 L CNN
 F 1 "SiS402DN" H 6454 1905 50  0000 L CNN
 F 2 "Package_SO:Vishay_PowerPAK_1212-8_Single" H 6250 2450 50  0001 C CNN
@@
 AR Path="/6202E846/6236E79F" Ref="#PWR029"  Part="1"
 AR Path="/620593AE/6236E79F" Ref="#PWR035"  Part="1"
-F 0 "#PWR035" H 6350 1900 50  0001 C CNN
+F 0 "#PWR029" H 6350 1900 50  0001 C CNN
 F 1 "GND" H 6355 1977 50  0000 C CNN
 F 2 "" H 6350 2150 50  0001 C CNN

Commit message: exposed NRST
Changed lines of the file:
@@
 AR Path="/61C031A1/61C0AE1D" Ref="#PWR?"  Part="1"
 AR Path="/61C031A3/61C0AE1D" Ref="#PWR?"  Part="1"
-AR Path="/6202E846/61C0AE1D" Ref="#PWR031"  Part="1"
-AR Path="/620593AE/61C0AE1D" Ref="#PWR037"  Part="1"
-F 0 "#PWR031" H 3000 2400 50  0001 C CNN
+AR Path="/6202E846/61C0AE1D" Ref="#PWR030"  Part="1"
+AR Path="/620593AE/61C0AE1D" Ref="#PWR036"  Part="1"
+F 0 "#PWR036" H 3000 2400 50  0001 C CNN
 F 1 "GND" H 3005 2477 50  0000 C CNN
 F 2 "" H 3000 2650 50  0001 C CNN
@@
 AR Path="/6202E846/61C0ECF9" Ref="R12"  Part="1"
 AR Path="/620593AE/61C0ECF9" Ref="R14"  Part="1"
-F 0 "R12" H 1530 2646 50  0000 R CNN
+F 0 "R14" H 1530 2646 50  0000 R CNN
 F 1 "4.7k" H 1530 2555 50  0000 R CNN
 F 2 "Resistor_SMD:R_0402_1005Metric" V 1530 2600 50  0001 C CNN
@@
 AR Path="/61C031A1/61C1051F" Ref="#PWR?"  Part="1"
 AR Path="/61C031A3/61C1051F" Ref="#PWR?"  Part="1"
-AR Path="/6202E846/61C1051F" Ref="#PWR032"  Part="1"
-AR Path="/620593AE/61C1051F" Ref="#PWR038"  Part="1"
-F 0 "#PWR032" H 1600 2500 50  0001 C CNN
+AR Path="/6202E846/61C1051F" Ref="#PWR031"  Part="1"
+AR Path="/620593AE/61C1051F" Ref="#PWR037"  Part="1"
+F 0 "#PWR037" H 1600 2500 50  0001 C CNN
 F 1 "GND" H 1605 2577 50  0000 C CNN
 F 2 "" H 1600 2750 50  0001 C CNN
@@
 AR Path="/6202E846/61C0A1BB" Ref="Q1"  Part="1"
 AR Path="/620593AE/61C0A1BB" Ref="Q5"  Part="1"
-F 0 "Q1" H 3091 1496 50  0000 L CNN
+F 0 "Q5" H 3091 1496 50  0000 L CNN
 F 1 "MMBT5551" H 3091 1405 50  0000 L CNN
 F 2 "Package_TO_SOT_SMD:SOT-23" H 3100 1375 50  0001 L CIN
@@
 AR Path="/6202E846/61C5A1AF" Ref="R11"  Part="1"
 AR Path="/620593AE/61C5A1AF" Ref="R13"  Part="1"
-F 0 "R11" V 3657 1950 50  0000 C CNN
+F 0 "R13" V 3657 1950 50  0000 C CNN
 F 1 "100" V 3566 1950 50  0000 C CNN
 F 2 "Resistor_SMD:R_0402_1005Metric_Pad0.72x0.64mm_HandSolder" V 3380 1950 50  0001 C CNN
@@
 AR Path="/6202E846/61C4E023" Ref="Q4"  Part="1"
 AR Path="/620593AE/61C4E023" Ref="Q8"  Part="1"
-F 0 "Q4" H 3091 2404 50  0000 L CNN
+F 0 "Q8" H 3091 2404 50  0000 L CNN
 F 1 "MMBT5401" H 3091 2495 50  0000 L CNN
 F 2 "Package_TO_SOT_SMD:SOT-23" H 3100 2550 50  0001 C CNN
@@
 AR Path="/6202E846/61D142B7" Ref="C10"  Part="1"
 AR Path="/620593AE/61D142B7" Ref="C12"  Part="1"
-F 0 "C10" H 1265 1346 50  0000 L CNN
+F 0 "C12" H 1265 1346 50  0000 L CNN
 F 1 "100n" H 1265 1255 50  0000 L CNN
 F 2 "Capacitor_SMD:C_0402_1005Metric" H 1188 1150 50  0001 C CNN
@@
 AR Path="/61C031A1/61D15BBF" Ref="#PWR?"  Part="1"
 AR Path="/61C031A3/61D15BBF" Ref="#PWR?"  Part="1"
-AR Path="/6202E846/61D15BBF" Ref="#PWR027"  Part="1"
-AR Path="/620593AE/61D15BBF" Ref="#PWR033"  Part="1"
-F 0 "#PWR027" H 1150 1200 50  0001 C CNN
+AR Path="/6202E846/61D15BBF" Ref="#PWR026"  Part="1"
+AR Path="/620593AE/61D15BBF" Ref="#PWR032"  Part="1"
+F 0 "#PWR032" H 1150 1200 50  0001 C CNN
 F 1 "GND" H 1155 1277 50  0000 C CNN
 F 2 "" H 1150 1450 50  0001 C CNN
@@
 AR Path="/6202E846/622D62B8" Ref="Q2"  Part="1"
 AR Path="/620593AE/622D62B8" Ref="Q6"  Part="1"
-F 0 "Q2" H 5304 1996 50  0000 L CNN
+F 0 "Q6" H 5304 1996 50  0000 L CNN
 F 1 "SiS402DN" H 5304 1905 50  0000 L CNN
 F 2 "Package_SO:Vishay_PowerPAK_1212-8_Single" H 5100 2450 50  0001 C CNN
@@
 AR Path="/61C031A3/6203BB32" Ref="#PWR?"  Part="1"
 AR Path="/6203BB32" Ref="#PWR?"  Part="1"
-AR Path="/6202E846/6203BB32" Ref="#PWR028"  Part="1"
-AR Path="/620593AE/6203BB32" Ref="#PWR034"  Part="1"
-F 0 "#PWR028" H 5200 1900 50  0001 C CNN
+AR Path="/6202E846/6203BB32" Ref="#PWR027"  Part="1"
+AR Path="/620593AE/6203BB32" Ref="#PWR033"  Part="1"
+F 0 "#PWR033" H 5200 1900 50  0001 C CNN
 F 1 "GND" H 5205 1977 50  0000 C CNN
 F 2 "" H 5200 2150 50  0001 C CNN
@@
 AR Path="/6202E846/61C61D09" Ref="C11"  Part="1"
 AR Path="/620593AE/61C61D09" Ref="C13"  Part="1"
-F 0 "C11" H 4035 2146 50  0000 R CNN
+F 0 "C13" H 4035 2146 50  0000 R CNN
 F 1 "100n" H 4035 2055 50  0000 R CNN
 F 2 "Capacitor_SMD:C_0402_1005Metric_Pad0.74x0.62mm_HandSolder" H 4188 1950 50  0001 C CNN
@@
 AR Path="/61C031A1/61C20664" Ref="#PWR?"  Part="1"
 AR Path="/61C031A3/61C20664" Ref="#PWR?"  Part="1"
-AR Path="/6202E846/61C20664" Ref="#PWR030"  Part="1"
-AR Path="/620593AE/61C20664" Ref="#PWR036"  Part="1"
-F 0 "#PWR030" H 4150 2000 50  0001 C CNN
+AR Path="/6202E846/61C20664" Ref="#PWR029"  Part="1"
+AR Path="/620593AE/61C20664" Ref="#PWR035"  Part="1"
+F 0 "#PWR035" H 4150 2000 50  0001 C CNN
 F 1 "GND" H 4155 2077 50  0000 C CNN
 F 2 "" H 4150 2250 50  0001 C CNN
@@
 AR Path="/6202E846/6236D64F" Ref="Q3"  Part="1"
 AR Path="/620593AE/6236D64F" Ref="Q7"  Part="1"
-F 0 "Q3" H 6454 1996 50  0000 L CNN
+F 0 "Q7" H 6454 1996 50  0000 L CNN
 F 1 "SiS402DN" H 6454 1905 50  0000 L CNN
 F 2 "Package_SO:Vishay_PowerPAK_1212-8_Single" H 6250 2450 50  0001 C CNN
@@
 AR Path="/61C031A3/6236E79F" Ref="#PWR?"  Part="1"
 AR Path="/6236E79F" Ref="#PWR?"  Part="1"
-AR Path="/6202E846/6236E79F" Ref="#PWR029"  Part="1"
-AR Path="/620593AE/6236E79F" Ref="#PWR035"  Part="1"
-F 0 "#PWR029" H 6350 1900 50  0001 C CNN
+AR Path="/6202E846/6236E79F" Ref="#PWR028"  Part="1"
+AR Path="/620593AE/6236E79F" Ref="#PWR034"  Part="1"
+F 0 "#PWR034" H 6350 1900 50  0001 C CNN
 F 1 "GND" H 6355 1977 50  0000 C CNN
 F 2 "" H 6350 2150 50  0001 C CNN
